Commit message: Add URDF and Xacro files for DFRbot, including base and road wheel definitions

File: src/robo_description/urdf/DFRbot.urdf.xacro (robot description, xacro)
@@ -1,4 +1,10 @@
 <?xml version='1.0' encoding='utf-8'?>
-<robot name="DFRbot">
+<robot xmlns:xacro="http://www.ros.org/wiki/xacro">
+    <material name="metal_black">
+        <color rgba="0.0 0.0 0.0 1.0" />
+    </material>
+    <material name="road_wheel">
+        <color rgba="0.957 0.839 0.576 1.0" />
+    </material>
     <link name="base_link">
         <inertial>
@@ -14,4 +20,5 @@
                 <mesh filename="../meshes/base_link.stl" scale="0.001 0.001 0.001" />
             </geometry>
+            <material name="metal_black" />
         </visual>
         <collision name="base_link_collision">
